File: Hardware/sunrise-alarm/sunrise-alarm.kicad_sch (KiCad schematic)
At the start: 54 parts, among them IC1 CD74HC237M96, IC2 ACST410-8BTR, J1 Conn_01x08_Male, J2 Conn_01x06_Female, J3 Conn_01x06_Male, J4 Conn_01x05, J6 Conn_Socket, P1 Conn_WallPlug, Q1 2N3904, SW1 SW_Push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

Commit message: Replaced generic button.
Parts:
- removed SW1: SW_Push, symbol Switch:SW_Push
- added S?: PTS526_SK15_SMTR2_LFS, PTS526SK15SMTR2LFS, symbol Custom:PTS526_SK15_SMTR2_LFS
Connections:
- net GND: now also S?.1
- net at JP1.2 (B), R1.2, R2.1: now also S?.4
Changed lines of the file:
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@@
+    (stroke (width 0) (type default) (color 0 0 0 0))
+  )
+  (wire (pts (xy 35.56 123.19) (xy 38.1 123.19))
     (stroke (width 0) (type default) (color 0 0 0 0))
   )
@@
     (stroke (width 0) (type default) (color 0 0 0 0))
   )
+  (wire (pts (xy 17.78 123.19) (xy 20.32 123.19))
+    (stroke (width 0) (type default) (color 0 0 0 0))
+  )
   (wire (pts (xy 41.91 17.78) (xy 41.91 20.32))
     (stroke (width 0) (type default) (color 0 0 0 0))
@@
   )
   (wire (pts (xy 270.51 100.33) (xy 274.32 100.33))
-    (stroke (width 0) (type default) (color 0 0 0 0))
-  )
-  (wire (pts (xy 38.1 123.19) (xy 27.94 123.19))
     (stroke (width 0) (type default) (color 0 0 0 0))
   )
@@
     (pin "2")
   )
-  (symbol (lib_id "Switch:SW_Push") (at 22.86 123.19 0) (unit 1)
-    (in_bom yes) (on_board yes)
-    (property "Reference" "SW1" (id 0) (at 22.86 115.951 0))
-    (property "Value" "SW_Push" (id 1) (at 22.86 118.2624 0))
-    (property "Footprint" "" (id 2) (at 22.86 118.11 0)
-      (effects (font (size 1.27 1.27)) hide)
-    )
-    (property "Datasheet" "~" (id 3) (at 22.86 118.11 0)
-      (effects (font (size 1.27 1.27)) hide)
-    )
-    (pin "1")
-    (pin "2")
-  )
   (symbol (lib_id "Device:C") (at 22.86 144.78 0) (unit 1)
     (in_bom yes) (on_board yes)
@@
     (pin "2")
   )
+  (symbol (lib_id "Custom:PTS526_SK15_SMTR2_LFS") (at 12.7 123.19 0) (unit 1)
+    (in_bom yes) (on_board yes)
+    (property "Reference" "S?" (id 0) (at 27.94 115.57 0))
+    (property "Value" "PTS526_SK15_SMTR2_LFS" (id 1) (at 27.94 118.11 0))
+    (property "Footprint" "PTS526SK15SMTR2LFS" (id 2) (at 39.37 120.65 0)
+      (effects (font (size 1.27 1.27)) (justify left) hide)
+    )
+    (property "Datasheet" "https://www.ckswitches.com/media/2780/pts526.pdf" (id 3) (at 39.37 123.19 0)
+      (effects (font (size 1.27 1.27)) (justify left) hide)
+    )
+    (property "Description" "Tact 5.2 x 5.2, 1.5 mm H, 260gf, G leads, No ground pin, metal actuator" (id 4) (at 39.37 125.73 0)
+      (effects (font (size 1.27 1.27)) (justify left) hide)
+    )
+    (property "Height" "1.65" (id 5) (at 39.37 128.27 0)
+      (effects (font (size 1.27 1.27)) (justify left) hide)
+    )
+    (property "Mouser Part Number" "611-PTS526SK15SMR2L" (id 6) (at 39.37 130.81 0)
+      (effects (font (size 1.27 1.27)) (justify left) hide)
+    )
+    (property "Mouser Price/Stock" "https://www.mouser.co.uk/ProductDetail/CK/PTS526-SK15-SMTR2-LFS?qs=UXgszm6BlbF5Ezp94JAQtw%3D%3D" (id 7) (at 39.37 133.35 0)
+      (effects (font (size 1.27 1.27)) (justify left) hide)
+    )
+    (property "Manufacturer_Name" "C & K COMPONENTS" (id 8) (at 39.37 135.89 0)
+      (effects (font (size 1.27 1.27)) (justify left) hide)
+    )
+    (property "Manufacturer_Part_Number" "PTS526 SK15 SMTR2 LFS" (id 9) (at 39.37 138.43 0)
+      (effects (font (size 1.27 1.27)) (justify left) hide)
+    )
+    (pin "1")
+    (pin "2")
+    (pin "3")
+    (pin "4")
+  )
   (symbol (lib_id "Device:C_Polarized_Small") (at 22.86 85.09 0) (mirror y) (unit 1)
     (in_bom yes) (on_board yes) (fields_autoplaced)
@@
       (reference "S2") (unit 1) (value "PTS526_SK15_SMTR2_LFS") (footprint "PTS526SK15SMTR2LFS")
     )
-    (path "/00000000-0000-0000-0000-0000617c3584"
-      (reference "SW1") (unit 1) (value "SW_Push") (footprint "")
+    (path "/ba1faa34-4cd5-4b9e-a01e-497b4ce030cf"
+      (reference "S?") (unit 1) (value "PTS526_SK15_SMTR2_LFS") (footprint "PTS526SK15SMTR2LFS")
     )
     (path "/dcd57494-6b7e-4b45-84f4-4423ca227cf9"
